File: PCB/SCARTiera.kicad_pcb (KiCad board)
At the start: 2 copper layers, 214 x 123 mm, 25 parts, among them J1 SCART-F, J2 SCART-F, J3 SCART-F, J4 SCART-TV, J5 SCART-F, J6 SCART-F, J7 SCART-F, SW1 SW_DIP_x09, SW2 SW_DIP_x09, SW3 SW_DIP_x09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

Commit message: Add files via upload
Parts:
- moved SW1 0.50 mm to (89.0, 140.5)
Other:
- outline, holes or cut-outs redrawn
- board text added: "1"
- board text added: "2"
- board text added: "3"
- board text added: "4"
- board text added: "5"
- board text added: "6"
- board text added: "TV"
Changed lines of the file:
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@@
 			(drillshape 0)
 			(scaleselection 1)
-			(outputdirectory "../Gerber/")
+			(outputdirectory "Gerbers/")
 		)
 	)
@@
 	(footprint "InterlockSwitch_18pin:Switch"
 		(layer "F.Cu")
-		(at 89.5 140.5)
+		(at 89 140.5)
 		(property "Reference" "SW1"
 			(at -2 10.25 0)
@@
 		(embedded_fonts no)
 	)
+	(gr_circle
+		(center 227.5 162)
+		(end 229.5 159.5)
+		(stroke
+			(width 0.05)
+			(type default)
+		)
+		(fill no)
+		(layer "Edge.Cuts")
+	)
+	(gr_circle
+		(center 226 54)
+		(end 228.5 52)
+		(stroke
+			(width 0.05)
+			(type default)
+		)
+		(fill no)
+		(layer "Edge.Cuts")
+	)
+	(gr_circle
+		(center 29.5 55)
+		(end 31.5 52.5)
+		(stroke
+			(width 0.05)
+			(type default)
+		)
+		(fill no)
+		(layer "Edge.Cuts")
+	)
 	(gr_rect
 		(start 21 46.5)
@@
 		(layer "Edge.Cuts")
 	)
+	(gr_circle
+		(center 29.5 159)
+		(end 31.5 156.5)
+		(stroke
+			(width 0.05)
+			(type default)
+		)
+		(fill no)
+		(layer "Edge.Cuts")
+	)
+	(gr_text "5"
+		(at 137.5 161 0)
+		(layer "F.SilkS")
+		(effects
+			(font
+				(size 5 5)
+				(thickness 0.625)
+			)
+			(justify left bottom)
+		)
+	)
+	(gr_text "4\n"
+		(at 122.5 161 0)
+		(layer "F.SilkS")
+		(effects
+			(font
+				(size 5 5)
+				(thickness 0.625)
+			)
+			(justify left bottom)
+		)
+	)
+	(gr_text "6"
+		(at 153 161 0)
+		(layer "F.SilkS")
+		(effects
+			(font
+				(size 5 5)
+				(thickness 0.625)
+			)
+			(justify left bottom)
+		)
+	)
+	(gr_text "TV"
+		(at 215 131.5 0)
+		(layer "F.SilkS")
+		(effects
+			(font
+				(size 5 5)
+				(thickness 0.625)
+			)
+			(justify left bottom)
+		)
+	)
+	(gr_text "4\n"
+		(at 139 127 0)
+		(layer "F.SilkS")
+		(effects
+			(font
+				(size 5 5)
+				(thickness 0.625)
+			)
+			(justify left bottom)
+		)
+	)
+	(gr_text "3\n"
+		(at 107.5 161 0)
+		(layer "F.SilkS")
+		(effects
+			(font
+				(size 5 5)
+				(thickness 0.625)
+			)
+			(justify left bottom)
+		)
+	)
+	(gr_text "2"
+		(at 93 161 0)
+		(layer "F.SilkS")
+		(effects
+			(font
+				(size 5 5)
+				(thickness 0.625)
+			)
+			(justify left bottom)
+		)
+	)
+	(gr_text "5"
+		(at 167 127 0)
+		(layer "F.SilkS")
+		(effects
+			(font
+				(size 5 5)
+				(thickness 0.625)
+			)
+			(justify left bottom)
+		)
+	)
+	(gr_text "3\n"
+		(at 111 127 0)
+		(layer "F.SilkS")
+		(effects
+			(font
+				(size 5 5)
+				(thickness 0.625)
+			)
+			(justify left bottom)
+		)
+	)
+	(gr_text "6"
+		(at 197 127 0)
+		(layer "F.SilkS")
+		(effects
+			(font
+				(size 5 5)
+				(thickness 0.625)
+			)
+			(justify left bottom)
+		)
+	)
+	(gr_text "2"
+		(at 81.5 127 0)
+		(layer "F.SilkS")
+		(effects
+			(font
+				(size 5 5)
+				(thickness 0.625)
+			)
+			(justify left bottom)
+		)
+	)
+	(gr_text "1"
+		(at 78 161 0)
+		(layer "F.SilkS")
+		(effects
+			(font
+				(size 5 5)
+				(thickness 0.625)
+			)
+			(justify left bottom)
+		)
+	)
+	(gr_text "1"
+		(at 53 127 0)
+		(layer "F.SilkS")
+		(effects
+			(font
+				(size 5 5)
+				(thickness 0.625)
+			)
+			(justify left bottom)
+		)
+	)
 	(segment
 		(start 39.77 82.64)
@@
 	)
 	(segment
-		(start 85.142446 132.949)
-		(end 88.949 136.755554)
+		(start 86 138.5)
+		(end 90 142.5)
 		(width 0.2)
 		(layer "F.Cu")
@@
 	)
 	(segment
-		(start 88.949 140.949)
-		(end 90.5 142.5)
+		(start 50.3819 132.949)
+		(end 85 132.949)
 		(width 0.2)
 		(layer "F.Cu")
@@
 	)
 	(segment
-		(start 50.3819 132.949)
-		(end 85.142446 132.949)
+		(start 85 132.949)
+		(end 86 133.949)
+		(width 0.2)
+		(layer "F.Cu")
+		(net 16)
+	)
+	(segment
+		(start 86 133.949)
+		(end 86 138.5)
 		(width 0.2)
 		(layer "F.Cu")
@@
 		(width 0.2)
 		(layer "F.Cu")
-		(net 16)
-	)
-	(segment
-		(start 88.949 136.755554)
-		(end 88.949 140.949)
-		(width 0.2)
-		(layer "F.Cu")

Commit message: Add files via upload
Routing:
- added copper zone on B.Cu, net GND
Changed lines of the file:
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@@
 			(pinfunction "P4")
 			(pintype "passive")
+			(zone_connect 2)
 		)
 		(pad "5" thru_hole oval
@@
 			(pinfunction "P5")
 			(pintype "passive")
+			(zone_connect 2)
 		)
 		(pad "6" thru_hole oval
@@
 			(pinfunction "P9")
 			(pintype "passive")
+			(zone_connect 2)
 		)
 		(pad "10" thru_hole oval
@@
 			(pinfunction "P13")
 			(pintype "passive")
+			(zone_connect 2)
 		)
 		(pad "14" thru_hole oval
@@
 			(pinfunction "P17")
 			(pintype "passive")
+			(zone_connect 2)
 		)
 		(pad "18" thru_hole oval
@@
 			(pinfunction "P18")
 			(pintype "passive")
+			(zone_connect 2)
 		)
 		(pad "19" thru_hole oval
@@
 			(pinfunction "P21")
 			(pintype "passive")
+			(zone_connect 2)
 		)
 		(embedded_fonts no)
@@
 			(pinfunction "P4")
 			(pintype "passive")
+			(zone_connect 2)
 		)
 		(pad "5" thru_hole oval
@@
 			(pinfunction "P5")
 			(pintype "passive")
+			(zone_connect 2)
 		)
 		(pad "6" thru_hole oval
@@
 			(pinfunction "P9")
 			(pintype "passive")
+			(zone_connect 2)
 		)
 		(pad "10" thru_hole oval
@@
 			(pinfunction "P13")
 			(pintype "passive")
+			(zone_connect 2)
 		)
 		(pad "14" thru_hole oval
@@
 			(pinfunction "P17")
 			(pintype "passive")
+			(zone_connect 2)
 		)
 		(pad "18" thru_hole oval
@@
 			(pinfunction "P18")
 			(pintype "passive")
+			(zone_connect 2)
 		)
 		(pad "19" thru_hole oval
@@
 			(pinfunction "P21")
 			(pintype "passive")
+			(zone_connect 2)
 		)
 		(embedded_fonts no)
@@
 			(pinfunction "P4")
 			(pintype "passive")
+			(zone_connect 2)
 		)
 		(pad "5" thru_hole oval
@@
 			(pinfunction "P5")
 			(pintype "passive")
+			(zone_connect 2)
 		)
 		(pad "6" thru_hole oval
@@
 			(pinfunction "P9")
 			(pintype "passive")
+			(zone_connect 2)
 		)
 		(pad "10" thru_hole oval
@@
 			(pinfunction "P13")
 			(pintype "passive")
+			(zone_connect 2)
 		)
 		(pad "14" thru_hole oval
@@
 			(pinfunction "P17")
 			(pintype "passive")
+			(zone_connect 2)
 		)
 		(pad "18" thru_hole oval
@@
 			(pinfunction "P18")
 			(pintype "passive")
+			(zone_connect 2)
 		)
 		(pad "19" thru_hole oval
@@
 			(pinfunction "P21")
 			(pintype "passive")
+			(zone_connect 2)
 		)
 		(embedded_fonts no)
@@
 			(pinfunction "P4")
 			(pintype "passive")
+			(zone_connect 2)
 		)
 		(pad "5" thru_hole oval
@@
 			(pinfunction "P5")
 			(pintype "passive")
+			(zone_connect 2)
 		)
 		(pad "6" thru_hole oval
@@
 			(pinfunction "P9")
 			(pintype "passive")
+			(zone_connect 2)
 		)
 		(pad "10" thru_hole oval
@@
 			(pinfunction "P13")
 			(pintype "passive")
+			(zone_connect 2)
 		)
 		(pad "14" thru_hole oval
@@
 			(pinfunction "P17")
 			(pintype "passive")
+			(zone_connect 2)
 		)
 		(pad "18" thru_hole oval
@@
 			(pinfunction "P18")
 			(pintype "passive")
+			(zone_connect 2)
 		)
 		(pad "19" thru_hole oval
@@
 			(pinfunction "P21")
 			(pintype "passive")
+			(zone_connect 2)
 		)
 		(embedded_fonts no)
@@
 			(pinfunction "P4")
 			(pintype "passive")
+			(zone_connect 2)
 		)
 		(pad "5" thru_hole oval
@@
 			(pinfunction "P5")
 			(pintype "passive")
+			(zone_connect 2)
 		)
 		(pad "6" thru_hole oval
@@
 			(pinfunction "P9")
 			(pintype "passive")
+			(zone_connect 2)
 		)
 		(pad "10" thru_hole oval
@@
 			(pinfunction "P13")
 			(pintype "passive")
+			(zone_connect 2)
 		)
 		(pad "14" thru_hole oval
@@
 			(pinfunction "P17")
 			(pintype "passive")
+			(zone_connect 2)
 		)
 		(pad "18" thru_hole oval
@@
 			(pinfunction "P18")
 			(pintype "passive")
+			(zone_connect 2)
 		)
 		(pad "19" thru_hole oval
@@
 			(pinfunction "P21")
 			(pintype "passive")
+			(zone_connect 2)
 		)
 		(embedded_fonts no)
@@
 			(pinfunction "P4")
 			(pintype "passive")
+			(zone_connect 2)
 		)
 		(pad "5" thru_hole oval
@@
 			(pinfunction "P5")
 			(pintype "passive")
+			(zone_connect 2)
 		)
 		(pad "6" thru_hole oval
@@
 			(pinfunction "P9")
 			(pintype "passive")
+			(zone_connect 2)
 		)
 		(pad "10" thru_hole oval
@@
 			(pinfunction "P13")
 			(pintype "passive")
+			(zone_connect 2)
 		)
 		(pad "14" thru_hole oval
@@
 			(pinfunction "P17")
 			(pintype "passive")
+			(zone_connect 2)
 		)
 		(pad "18" thru_hole oval
@@
 			(pinfunction "P18")
 			(pintype "passive")
+			(zone_connect 2)
 		)
 		(pad "19" thru_hole oval
@@
 			(pinfunction "P21")
 			(pintype "passive")
+			(zone_connect 2)
 		)
 		(embedded_fonts no)
@@
 			(pinfunction "P4")
 			(pintype "passive")
+			(zone_connect 2)
 		)
 		(pad "5" thru_hole oval
@@
 			(pinfunction "P5")
 			(pintype "passive")
+			(zone_connect 2)
 		)
 		(pad "6" thru_hole oval
@@
 			(pinfunction "P9")
 			(pintype "passive")
+			(zone_connect 2)
 		)
 		(pad "10" thru_hole oval
@@
 			(pinfunction "P13")
 			(pintype "passive")
+			(zone_connect 2)
 		)
 		(pad "14" thru_hole oval
@@
 			(pinfunction "P17")
 			(pintype "passive")
+			(zone_connect 2)
 		)
 		(pad "18" thru_hole oval
@@
 			(pinfunction "P18")
 			(pintype "passive")
+			(zone_connect 2)
 		)
 		(pad "19" thru_hole oval
@@
 			(pinfunction "P21")
 			(pintype "passive")
+			(zone_connect 2)
 		)
 		(embedded_fonts no)
@@
 	)
 	(segment
-		(start 36 122)
-		(end 44.5 122)
-		(width 1)
-		(layer "B.Cu")
-		(net 3)
-	)
-	(segment
 		(start 113 111)
 		(end 113.5 111)
@@
 	)
 	(segment
-		(start 51 115.5)
-		(end 51 115)
-		(width 1)
-		(layer "B.Cu")
-		(net 3)
-	)
-	(segment
-		(start 51 115)
-		(end 55 111)
+		(start 36 122)
+		(end 44 122)
 		(width 1)
 		(layer "B.Cu")
@@
 	)
 	(segment
+		(start 29 115)
+		(end 36 122)
+		(width 1)
+		(layer "B.Cu")
+		(net 3)
+	)
+	(segment
 		(start 107 111)
 		(end 113 111)
@@
 	)
 	(segment
-		(start 79 111)
-		(end 84 111)
+		(start 44 122)
+		(end 55 111)
 		(width 1)
 		(layer "B.Cu")
@@
 	)
 	(segment
-		(start 203.62 97.88)
-		(end 216.5 97.88)
+		(start 29 112)
+		(end 29 115)
 		(width 1)
 		(layer "B.Cu")
@@
 	)
 	(segment
-		(start 141.5 111)
-		(end 152 121.5)
+		(start 79 111)
+		(end 84 111)
 		(width 1)
 		(layer "B.Cu")
@@
 	)
 	(segment
-		(start 29 112)
-		(end 29 115)
+		(start 203.62 97.88)
+		(end 216.5 97.88)
 		(width 1)
 		(layer "B.Cu")
@@
 	)
 	(segment
-		(start 134.5 111)
-		(end 141 111)
+		(start 141.5 111)
+		(end 152 121.5)
 		(width 1)
 		(layer "B.Cu")
@@
 	)
 	(segment
-		(start 44.5 122)
-		(end 51 115.5)
+		(start 134.5 111)
+		(end 141 111)
 		(width 1)
 		(layer "B.Cu")
@@
 	)
 	(segment
-		(start 29 115)
-		(end 36 122)
-		(width 1)
-		(layer "B.Cu")
-		(net 3)
-	)
-	(segment
 		(start 141 111)
 		(end 141.5 111)
@@
 		(start 39.77 75.02)
 		(end 42.955 75.02)
-		(width 0.2)
+		(width 0.5)
 		(layer "B.Cu")
 		(net 9)
@@
 		(start 44.85 76.915)
 		(end 47.415 76.915)
-		(width 0.2)
+		(width 0.5)
 		(layer "B.Cu")
 		(net 9)
@@
 		(start 44.85 92.155)
 		(end 47.845 92.155)
-		(width 0.2)
+		(width 0.5)
 		(layer "B.Cu")
 		(net 9)
@@
 		(start 44.85 84.535)
 		(end 47.965 84.535)
-		(width 0.2)
+		(width 0.5)
 		(layer "B.Cu")
 		(net 9)
@@
 		(start 39.77 101.69)
 		(end 42.935 101.69)
-		(width 0.2)
+		(width 0.5)
 		(layer "B.Cu")
 		(net 9)
@@
 		(start 42.935 101.69)
 		(end 44.85 99.775)
-		(width 0.2)
+		(width 0.5)
 		(layer "B.Cu")
 		(net 9)
@@
 		(start 42.955 75.02)
 		(end 44.85 76.915)
-		(width 0.2)
+		(width 0.5)
 		(layer "B.Cu")
 		(net 9)
@@
 		(start 44.85 99.775)
 		(end 47.775 99.775)
-		(width 0.2)
+		(width 0.5)
 		(layer "B.Cu")
 		(net 9)
@@
 		(net 99)
 	)
+	(zone
+		(net 9)
+		(net_name "GND")
+		(layer "B.Cu")
+		(hatch edge 0.5)
+		(connect_pads
+			(clearance 0.5)
+		)
+		(min_thickness 0.25)
+		(filled_areas_thickness no)
+		(fill yes
+			(thermal_gap 0.5)
+			(thermal_bridge_width 0.5)
+		)
+		(polygon
+			(pts
+				(xy 21 46.5) (xy 21 169.5) (xy 235 169.5) (xy 235 46.5)
+			)
+		)
+	)
 	(embedded_fonts no)

Commit message: Add files via upload
Parts:
- added REF**: MountingHole_3.2mm_M3, MountingHole:MountingHole_3.2mm_M3, F.Cu at (226.0, 54.0)
- added REF**: MountingHole_3.2mm_M3, MountingHole:MountingHole_3.2mm_M3, F.Cu at (29.5, 159.0)
- added REF**: MountingHole_3.2mm_M3, MountingHole:MountingHole_3.2mm_M3, F.Cu at (29.5, 55.0)
- added REF**: MountingHole_3.2mm_M3, MountingHole:MountingHole_3.2mm_M3, F.Cu at (227.5, 162.0)
Other:
- outline, holes or cut-outs redrawn
